Commit message: feat: Add camera to URDF, include joint state publisher, update RViz configuration, and add view_ws Makefile.

File: view_ws/src/car_description/urdf/car.urdf (robot description, URDF)
Before this commit: robot raspi_koma, 3 links, 2 joints
Links:
- added link camera_link; visual box size=0.01 0.04 0.01
Joints:
- added joint camera_joint: type fixed, parent base_link, child camera_link, origin xyz=0.09 0 0.02 rpy=0 0 0

Commit message: feat: Introduce front wheels and sonars to the car model, adjust camera origin, and refine RViz visualization.

File: view_ws/src/car_description/urdf/car.urdf (robot description, URDF)
Before this commit: robot raspi_koma, 4 links, 3 joints
Links:
- added link front_left_wheel; visual cylinder length=0.04 radius=0.035
- added link front_right_wheel; visual cylinder length=0.04 radius=0.035
- added link sonar_front_left; visual box size=0.01 0.02 0.01
- added link sonar_front_right; visual box size=0.01 0.02 0.01
Joints:
- added joint front_left_wheel_joint: type continuous, parent base_link, child front_left_wheel, origin xyz=0.05 0.08 0 rpy=0 0 0, axis 0 1 0
- added joint front_right_wheel_joint: type continuous, parent base_link, child front_right_wheel, origin xyz=0.05 -0.08 0 rpy=0 0 0, axis 0 1 0
- added joint sonar_front_left_joint: type fixed, parent base_link, child sonar_front_left, origin xyz=0.09 0.03 0 rpy=0 0 0
- added joint sonar_front_right_joint: type fixed, parent base_link, child sonar_front_right, origin xyz=0.09 -0.03 0 rpy=0 0 0
- joint camera_joint: origin xyz=0.09 0 0.02 rpy=0 0 0 -> xyz=0.06 0 0.02 rpy=0 0 0

Commit message: remove scripts and gazebo configuration

File: view_ws/src/car_description/urdf/car.urdf (robot description, URDF)
Before this commit: robot raspi_koma, 8 links, 7 joints
Links:
- link base_link: geometry visual box size=0.43 0.22 0.07
- link camera_link: geometry visual box size=0.02 0.05 0.03
- link front_left_wheel: geometry visual cylinder length=0.03 radius=0.035
- link front_right_wheel: geometry visual cylinder length=0.03 radius=0.035
- link left_wheel: geometry visual cylinder length=0.03 radius=0.035
- link right_wheel: geometry visual cylinder length=0.03 radius=0.035
Joints:
- joint camera_joint: origin xyz=0.06 0 0.02 rpy=0 0 0 -> xyz=0 0 0.035 rpy=0 0 0
- joint front_left_wheel_joint: origin xyz=0.05 0.08 0 rpy=0 0 0 -> xyz=0.095 0.13 -0.025 rpy=0 0 0
- joint front_right_wheel_joint: origin xyz=0.05 -0.08 0 rpy=0 0 0 -> xyz=0.095 -0.13 -0.025 rpy=0 0 0
- joint left_wheel_joint: origin xyz=-0.05 0.08 0 rpy=0 0 0 -> xyz=-0.145 0.13 -0.025 rpy=0 0 0
- joint right_wheel_joint: origin xyz=-0.05 -0.08 0 rpy=0 0 0 -> xyz=-0.145 -0.13 -0.025 rpy=0 0 0
- joint sonar_front_left_joint: origin xyz=0.09 0.03 0 rpy=0 0 0 -> xyz=0.215 0.045 -0.02 rpy=0 0 0.436
- joint sonar_front_right_joint: origin xyz=0.09 -0.03 0 rpy=0 0 0 -> xyz=0.215 -0.045 -0.02 rpy=0 0 -0.436

Commit message: update camera position

File: view_ws/src/car_description/urdf/car.urdf (robot description, URDF)
Before this commit: robot raspi_koma, 8 links, 7 joints
Joints:
- joint camera_joint: origin xyz=0 0 0.035 rpy=0 0 0 -> xyz=0.145 0 0.035 rpy=0 0 0

File: view_ws/src/car_description/urdf/raspikoma.urdf (robot description, URDF)
Before this commit: robot car, 3 links, 2 joints
Joints:
- joint camera_joint: origin xyz=0 0 0.035 rpy=0 0 0 -> xyz=0.145 0 0.035 rpy=0 0 0
